File: pcb/clockport.sch (KiCad schematic (older format))
At the start: 1 part

Commit message: hiererchy update
Changed lines of the file:
@@
 	1    0    0    -1
 $EndComp
-Wire Bus Line
-	1000 1000 1500 1000
-Wire Bus Line
-	1500 1000 5000 1000
-Connection ~ 1500 1000
 Entry Wire Line
 	1500 1500 1600 1600
@@
 Text Label 4500 2800 0    50   ~ 0
 A5
+Text HLabel 1000 1000 0    50   Input ~ 0
+TRPDR
+Text HLabel 1000 3000 0    50   Input ~ 0
+POWER_GND
 Wire Bus Line
-	1500 1000 1500 4000
+	1000 1000 1500 1000
+Connection ~ 1500 1000
+Wire Bus Line
+	1500 1000 5000 1000
+Wire Bus Line
+	1500 3000 1000 3000
+Wire Bus Line
+	1500 2400 1500 3000
+Wire Bus Line
+	1500 1000 1500 2200
 Wire Bus Line
 	5000 1000 5000 4000
-Text HLabel 1000 1000 0    50   Input ~ 0
-TRPDR
 $EndSCHEMATC
