File: pcb/trapdoor_connector.sch (KiCad schematic (older format))
At the start: 1 part, among them X1 A1200_trapdoor_connector

Commit message: buffer section finished, audio moved to expansion connector
Connections:
- net E_CLOCK: now reaches X1.100 (E_CLOCK)
- net CCKA: now reaches X1.117 (CCKA)
- net _RESET: now reaches X1.118 (_RESET)
Changed lines of the file:
@@
 Wire Bus Line
 	7900 3900 9750 3900
+Connection ~ 7900 3900
+Entry Wire Line
+	4900 1500 5000 1600
+Entry Wire Line
+	4900 1600 5000 1700
+Entry Wire Line
+	1000 5200 1100 5300
+Wire Wire Line
+	1100 5300 1550 5300
+Wire Wire Line
+	5000 1600 5450 1600
+Wire Wire Line
+	5450 1700 5000 1700
 Wire Bus Line
 	8400 600  8400 1400
@@
 Wire Bus Line
 	1000 700  1000 5800
-Connection ~ 7900 3900
+Text Label 5000 1600 0    50   ~ 0
+CCKA
+Text Label 5000 1700 0    50   ~ 0
+_RESET
+Text Label 1100 5300 0    50   ~ 0
+E_CLOCK
 $EndSCHEMATC
