File: pcb/WM1200.kicad_pcb (KiCad board)
At the start: 4 copper layers, 159 x 104 mm, 135 parts, among them Q1 BC817, Q2 BC817, Q3 BC817, Q4 BC817, Q5 BC817, Q6 BC817, U1 74LVCH162245A, U2 74LVCH162245A, U3 74LVCH162245A, U4 74LVCH162245A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

Commit message: Sync work
Routing:
- net +5VDC: track 0.00 -> 3.32 mm
Other:
- outline, holes or cut-outs redrawn
Changed lines of the file:
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@@
   (general
     (thickness 1.6)
-    (drawings 10)
-    (tracks 856)
+    (drawings 9)
+    (tracks 857)
     (zones 0)
     (modules 135)
@@
     (last_trace_width 0.25)
     (trace_clearance 0.2)
-    (zone_clearance 0.3)
+    (zone_clearance 0.28)
     (zone_45_only no)
     (trace_min 0.2)
@@
     (effects (font (size 2 2) (thickness 0.15) italic))
   )
-  (gr_circle (center 240 140) (end 243 140) (layer Edge.Cuts) (width 0.12))
   (gr_line (start 249 150) (end 90 150) (layer Edge.Cuts) (width 0.05))
   (gr_line (start 249 74) (end 249 150) (layer Edge.Cuts) (width 0.05))
@@
   (segment (start 130.175 70) (end 130.175 68.225) (width 0.25) (layer F.Cu) (net 20))
   (segment (start 132.3 70) (end 130.175 70) (width 0.25) (layer F.Cu) (net 20))
+  (segment (start 105.69 100.53) (end 102.37 100.53) (width 0.25) (layer In2.Cu) (net 21))
   (segment (start 129.399999 125.725001) (end 129.425 125.7) (width 0.25) (layer F.Cu) (net 22))
   (segment (start 127.045001 125.725001) (end 129.399999 125.725001) (width 0.3) (layer F.Cu) (net 22))
@@
   (segment (start 107.685 104.25) (end 107.595 104.34) (width 0.25) (layer F.Cu) (net 100))
   (segment (start 118.3 104.25) (end 107.685 104.25) (width 0.25) (layer F.Cu) (net 100))
-  (via micro (at 118.05 105.25) (size 0.3) (drill 0.1) (layers F.Cu B.Cu) (net 101))
-  (segment (start 121.75 105.25) (end 118.05 105.25) (width 0.25) (layer B.Cu) (net 101))
-  (segment (start 106.76763 105.61) (end 105.69 105.61) (width 0.25) (layer F.Cu) (net 101))
-  (segment (start 109.020763 106.697001) (end 107.933762 105.61) (width 0.25) (layer F.Cu) (net 101))
-  (segment (start 107.933762 105.61) (end 106.76763 105.61) (width 0.25) (layer F.Cu) (net 101))
-  (segment (start 116.602999 106.697001) (end 109.020763 106.697001) (width 0.25) (layer F.Cu) (net 101))
-  (segment (start 118.05 105.25) (end 116.602999 106.697001) (width 0.25) (layer F.Cu) (net 101))
+  (segment (start 107.933762 105.61) (end 109.020763 106.697001) (width 0.25) (layer F.Cu) (net 101))
+  (segment (start 105.69 105.61) (end 107.933762 105.61) (width 0.25) (layer F.Cu) (net 101))
+  (segment (start 119.3 105.25) (end 121.75 105.25) (width 0.25) (layer B.Cu) (net 101))
+  (segment (start 109.020763 106.697001) (end 116.602999 106.697001) (width 0.25) (layer F.Cu) (net 101))
+  (segment (start 118.05 105.25) (end 119.3 105.25) (width 0.25) (layer F.Cu) (net 101))
+  (segment (start 116.602999 106.697001) (end 118.05 105.25) (width 0.25) (layer F.Cu) (net 101))
+  (via micro (at 119.3 105.25) (size 0.3) (drill 0.1) (layers F.Cu B.Cu) (net 101))
   (segment (start 121 105.75) (end 121.75 105.75) (width 0.25) (layer B.Cu) (net 102))
   (segment (start 110.71763 105.75) (end 121 105.75) (width 0.25) (layer B.Cu) (net 102))
@@
   (segment (start 120.3 69) (end 118.3 69) (width 0.25) (layer F.Cu) (net 318))
   (zone (net 2) (net_name GND) (layer In1.Cu) (hatch edge 0.508)
-    (connect_pads (clearance 0.3))
+    (connect_pads (clearance 0.28))
     (min_thickness 0.2)
-    (fill yes (arc_segments 32) (thermal_gap 0.25) (thermal_bridge_width 0.3))
+    (fill (arc_segments 32) (thermal_gap 0.29) (thermal_bridge_width 0.3))
     (polygon
       (pts
@@
   )
   (zone (net 21) (net_name +5VDC) (layer In2.Cu) (hatch edge 0.508)
-    (connect_pads (clearance 0.3))
+    (connect_pads (clearance 0.28))
     (min_thickness 0.2)
-    (fill yes (arc_segments 32) (thermal_gap 0.25) (thermal_bridge_width 0.3))
+    (fill (arc_segments 32) (thermal_gap 0.29) (thermal_bridge_width 0.3))
     (polygon
       (pts

Commit message: some work on hdmi part
Parts:
- removed XT22, XT25: testpoint_cutline, WM1200:testpoint_cutline
- moved R22 21.1 mm to (217.8, 106.3), turned to 90 degrees
- moved R24 17.4 mm to (241.0, 96.2), turned to 180 degrees
- moved C22 15.4 mm to (241.0, 97.7), turned to 180 degrees
- moved C19 13.2 mm to (231.8, 109.9)
- moved R21 10.4 mm to (220.7, 101.8), turned to 90 degrees
- moved U7 8.47 mm to (226.2, 106.0)
- moved C21 6.48 mm to (231.1, 100.7), turned to 90 degrees
- moved R23 3.44 mm to (223.3, 112.0), turned to 270 degrees
- moved C20 3.30 mm to (220.5, 108.9), turned to 180 degrees
- moved R25 3.13 mm to (220.7, 106.3), turned to 90 degrees
Connections:
- U5 pad 35: Net-(U5-Pad35) -> _DSACK0
- U5 pad 36: Net-(U5-Pad36) -> _DSACK1
Routing:
- net +3V3_BUFFER: track 0.00 -> 140.8 mm, vias 0 -> 2
- net Net-(C22-Pad1): track 0.00 -> 30.8 mm
- net GND: track 69.3 -> 94.0 mm, vias 7 -> 21
- net Net-(U7-Pad7): track 0.00 -> 17.9 mm
- net Net-(U7-Pad8): track 0.00 -> 17.6 mm
- net Net-(U7-Pad9): track 0.00 -> 17.5 mm
- net Net-(U7-Pad10): track 0.00 -> 17.0 mm
- net Net-(C19-Pad1): track 0.00 -> 10.9 mm, vias 0 -> 2
- net FPGA_HDMI_CLK-: track 0.00 -> 9.61 mm
- net FPGA_HDMI_D2-: track 0.00 -> 9.59 mm
- net FPGA_HDMI_D1+: track 0.00 -> 9.54 mm
- net FPGA_HDMI_D0+: track 0.00 -> 9.38 mm
- net FPGA_HDMI_D0-: track 0.00 -> 9.34 mm
- net FPGA_HDMI_CLK+: track 0.00 -> 9.30 mm
- net FPGA_HDMI_D2+: track 0.00 -> 9.27 mm
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- added copper zone on In2.Cu, net +3V3_BUFFER
- added copper zone on In2.Cu, net FPGA_VCC3V3

Commit message: some more work done
Connections:
- U1 pad 26: FPGA_D24 -> Net-(U1-Pad26)
- U1 pad 27: FPGA_D25 -> Net-(U1-Pad27)
- U1 pad 29: FPGA_D26 -> Net-(U1-Pad29)
- U1 pad 30: FPGA_D27 -> Net-(U1-Pad30)
- U1 pad 32: FPGA_D28 -> Net-(U1-Pad32)
- U1 pad 33: FPGA_D29 -> Net-(U1-Pad33)
- U1 pad 35: FPGA_D30 -> Net-(U1-Pad35)
- U1 pad 36: FPGA_D31 -> Net-(U1-Pad36)
- U1 pad 37: FPGA_A7 -> Net-(U1-Pad37)
- U1 pad 38: FPGA_A6 -> Net-(U1-Pad38)
- U1 pad 40: FPGA_A5 -> Net-(U1-Pad40)
- U1 pad 41: FPGA_A4 -> Net-(U1-Pad41)
- U1 pad 43: FPGA_A3 -> Net-(U1-Pad43)
- U1 pad 44: FPGA_A2 -> Net-(U1-Pad44)
- U1 pad 46: FPGA_A1 -> Net-(U1-Pad46)
- U1 pad 47: FPGA_A0 -> Net-(U1-Pad47)
- U2 pad 26: FPGA_D8 -> Net-(U2-Pad26)
- U2 pad 27: FPGA_D9 -> Net-(U2-Pad27)
- U2 pad 29: FPGA_D10 -> Net-(U2-Pad29)
- U2 pad 30: FPGA_D11 -> Net-(U2-Pad30)
- U2 pad 32: FPGA_D12 -> Net-(U2-Pad32)
- U2 pad 33: FPGA_D13 -> Net-(U2-Pad33)
- U2 pad 35: FPGA_D14 -> Net-(U2-Pad35)
- U2 pad 36: FPGA_D15 -> Net-(U2-Pad36)
- U2 pad 37: FPGA_D16 -> Net-(U2-Pad37)
- U2 pad 38: FPGA_D17 -> Net-(U2-Pad38)
- U2 pad 40: FPGA_D18 -> Net-(U2-Pad40)
- U2 pad 41: FPGA_D19 -> Net-(U2-Pad41)
- U2 pad 43: FPGA_D20 -> Net-(U2-Pad43)
- U2 pad 44: FPGA_D21 -> Net-(U2-Pad44)
- U2 pad 46: FPGA_D22 -> Net-(U2-Pad46)
- U2 pad 47: FPGA_D23 -> Net-(U2-Pad47)
- U3 pad 26: FPGA_A8 -> Net-(U3-Pad26)
- U3 pad 27: FPGA_A9 -> Net-(U3-Pad27)
- U3 pad 29: FPGA_A10 -> Net-(U3-Pad29)
- U3 pad 30: FPGA_A11 -> Net-(U3-Pad30)
- U3 pad 32: FPGA_A12 -> Net-(U3-Pad32)
- U3 pad 33: FPGA_A13 -> Net-(U3-Pad33)
- U3 pad 35: FPGA_A14 -> Net-(U3-Pad35)
- U3 pad 36: FPGA_A15 -> Net-(U3-Pad36)
- U3 pad 37: FPGA_A16 -> Net-(U3-Pad37)
- U3 pad 38: FPGA_A17 -> Net-(U3-Pad38)
- U3 pad 40: FPGA_A18 -> Net-(U3-Pad40)
- U3 pad 41: FPGA_A19 -> Net-(U3-Pad41)
- U3 pad 43: FPGA_A20 -> Net-(U3-Pad43)
- U3 pad 44: FPGA_A21 -> Net-(U3-Pad44)
- U3 pad 46: FPGA_A22 -> Net-(U3-Pad46)
- U3 pad 47: FPGA_A23 -> Net-(U3-Pad47)
- U4 pad 26: FPGA_D7 -> Net-(U4-Pad26)
- U4 pad 27: FPGA_D6 -> Net-(U4-Pad27)
- U4 pad 29: FPGA_D5 -> Net-(U4-Pad29)
- U4 pad 30: FPGA_D4 -> Net-(U4-Pad30)
- U4 pad 32: FPGA_D3 -> Net-(U4-Pad32)
- U4 pad 33: FPGA_D2 -> Net-(U4-Pad33)
- U4 pad 35: FPGA_D1 -> Net-(U4-Pad35)
- U4 pad 36: FPGA_D0 -> Net-(U4-Pad36)
- XT10 pad 2: FPGA_FC2 -> Net-(XT10-Pad2)
- XT12 pad 2: _FPGA_DS -> Net-(XT12-Pad2)
- XT14 pad 2: FPGA_R_W -> Net-(XT14-Pad2)
- XT16 pad 2: _FPGA_AS -> Net-(XT16-Pad2)
- XT18 pad 2: FPGA_SIZE1 -> Net-(XT18-Pad2)
- XT20 pad 2: FPGA_SIZE0 -> Net-(XT20-Pad2)
- XT38 pad 2: _FPGA_IPL1 -> Net-(XT38-Pad2)
- XT40 pad 2: _FPGA_IPL2 -> Net-(XT40-Pad2)
- XT42 pad 2: _FPGA_IPL0 -> Net-(XT42-Pad2)
- XT44 pad 2: _FPGA_RST -> Net-(XT44-Pad2)
- XT46 pad 2: _FPGA_HLT -> Net-(XT46-Pad2)
- XT48 pad 2: _FPGA_BERR -> Net-(XT48-Pad2)
- XT50 pad 2: FPGA_CPUCLK_A -> Net-(XT50-Pad2)
- XT52 pad 2: _FPGA_KBRESET -> Net-(XT52-Pad2)
- XT6 pad 2: FPGA_FC0 -> Net-(XT6-Pad2)
- XT8 pad 2: FPGA_FC1 -> Net-(XT8-Pad2)
Routing:
- net GND: track 94.0 -> 164.9 mm, vias 21 -> 63
- net +3V3_BUFFER: track 140.8 -> 151.7 mm, vias 2 -> 11
- net +3V3_DC_DC: track 6.23 -> 13.4 mm
- net FPGA_VCC3V3: track 3.32 -> 8.97 mm, vias 1 -> 2
- net A1: track 13.2 -> 15.5 mm
