File: pcb/WM1200.sch (KiCad schematic (older format))
At the start: 0 parts

Commit message: ready for production
Changed lines of the file:
@@
 $Descr A4 11693 8268
 encoding utf-8
-Sheet 1 11
+Sheet 1 10
 Title "Wishmaster 1200"
-Date ""
+Date "2020-03-16"
 Rev "ES1"
 Comp "Created by Konfusion in 2020"
@@
 $EndDescr
 $Sheet
-S 3500 2000 1500 500
-U 5E5B86AA
-F0 "Testpoints" 50
-F1 "testpoints.sch" 50
-$EndSheet
-$Sheet
 S 6000 1500 1450 500
