File: pcb/power.sch (KiCad schematic (older format))
At the start: 7 parts, among them U6 ADP2108AUJ-3.3

Commit message: more footprints assigned, caps added into open collector base circuit
Parts:
- C11: value 4.7uF -> 4.7uF 35V; footprint (none) -> Capacitor_SMD:C_1210_3225Metric_Pad1.42x2.65mm_HandSolder
- C12: value 10uF -> 10uF 35V; footprint (none) -> Capacitor_SMD:C_1210_3225Metric_Pad1.42x2.65mm_HandSolder
- L1: footprint (none) -> Inductor_SMD:L_0603_1608Metric_Pad1.05x0.95mm_HandSolder
Changed lines of the file:
@@
 P 3000 2350
 F 0 "C11" H 3115 2396 50  0000 L CNN
-F 1 "4.7uF" H 3115 2305 50  0000 L CNN
-F 2 "" H 3038 2200 50  0001 C CNN
+F 1 "4.7uF 35V" H 3115 2305 50  0000 L CNN
+F 2 "Capacitor_SMD:C_1210_3225Metric_Pad1.42x2.65mm_HandSolder" H 3038 2200 50  0001 C CNN
 F 3 "~" H 3000 2350 50  0001 C CNN
 	1    3000 2350
@@
 P 5000 2350
 F 0 "C12" H 5115 2396 50  0000 L CNN
-F 1 "10uF" H 5115 2305 50  0000 L CNN
-F 2 "" H 5038 2200 50  0001 C CNN
+F 1 "10uF 35V" H 5115 2305 50  0000 L CNN
+F 2 "Capacitor_SMD:C_1210_3225Metric_Pad1.42x2.65mm_HandSolder" H 5038 2200 50  0001 C CNN
 F 3 "~" H 5000 2350 50  0001 C CNN
 	1    5000 2350
@@
 F 0 "L1" V 4590 2000 50  0000 C CNN
 F 1 "1uH" V 4499 2000 50  0000 C CNN
-F 2 "" H 4400 2000 50  0001 C CNN
+F 2 "Inductor_SMD:L_0603_1608Metric_Pad1.05x0.95mm_HandSolder" H 4400 2000 50  0001 C CNN
 F 3 "~" H 4400 2000 50  0001 C CNN
 	1    4400 2000

Commit message: working on pcb
Parts:
- JP1: footprint Connector_PinSocket_2.54mm:PinSocket_1x03_P2.54mm_Vertical -> Connector_PinHeader_2.54mm:PinHeader_1x03_P2.54mm_Vertical
- JP2: footprint Connector_PinSocket_2.54mm:PinSocket_1x02_P2.54mm_Vertical -> Connector_PinHeader_2.54mm:PinHeader_1x02_P2.54mm_Vertical
Changed lines of the file:
@@
 F 0 "JP1" V 3854 3602 50  0000 L CNN
 F 1 "Jumper_NC_Dual" V 3945 3602 50  0000 L CNN
-F 2 "Connector_PinSocket_2.54mm:PinSocket_1x03_P2.54mm_Vertical" H 3900 3500 50  0001 C CNN
+F 2 "Connector_PinHeader_2.54mm:PinHeader_1x03_P2.54mm_Vertical" H 3900 3500 50  0001 C CNN
 F 3 "~" H 3900 3500 50  0001 C CNN
 	1    3900 3500
@@
 F 0 "JP2" H 3900 4764 50  0000 C CNN
 F 1 "Jumper" H 3900 4673 50  0000 C CNN
-F 2 "Connector_PinSocket_2.54mm:PinSocket_1x02_P2.54mm_Vertical" H 3900 4500 50  0001 C CNN
+F 2 "Connector_PinHeader_2.54mm:PinHeader_1x02_P2.54mm_Vertical" H 3900 4500 50  0001 C CNN
 F 3 "~" H 3900 4500 50  0001 C CNN
 	1    3900 4500

Commit message: Buffers power scheme rework in progress, re-annotate board
Parts:
- renumbered C11 to C21, C12 to C22, XT55 to XT47
Changed lines of the file:
@@
 $EndComp
 $Comp
-L WM1200:testpoint_cutline XT55
+L WM1200:testpoint_cutline XT47
 U 1 1 5E716612
 P 2300 2050
-F 0 "XT55" H 2300 2233 50  0000 C CNN
+F 0 "XT47" H 2300 2233 50  0000 C CNN
 F 1 "testpoint_cutline" H 2300 2200 50  0001 C CNN
 F 2 "WM1200:testpoint_cutline" H 2450 2050 50  0001 C CNN
@@
 	3400 2000 3450 2000
 $Comp
-L Device:C C11
+L Device:C C21
 U 1 1 5E718DCB
 P 3000 2350
-F 0 "C11" H 3115 2396 50  0000 L CNN
+F 0 "C21" H 3115 2396 50  0000 L CNN
 F 1 "4.7uF 35V" H 3115 2305 50  0000 L CNN
 F 2 "Capacitor_SMD:C_1210_3225Metric_Pad1.42x2.65mm_HandSolder" H 3038 2200 50  0001 C CNN
@@
 	3000 2000 3400 2000
 $Comp
-L Device:C C12
+L Device:C C22
 U 1 1 5E71F97C
 P 5000 2350
-F 0 "C12" H 5115 2396 50  0000 L CNN
+F 0 "C22" H 5115 2396 50  0000 L CNN
 F 1 "10uF 35V" H 5115 2305 50  0000 L CNN
 F 2 "Capacitor_SMD:C_1210_3225Metric_Pad1.42x2.65mm_HandSolder" H 5038 2200 50  0001 C CNN

Commit message: still working
Parts:
- XT47: footprint WM1200:testpoint_cutline -> WM1200:testpoint_cutline_fat
Changed lines of the file:
@@
 F 0 "XT47" H 2300 2233 50  0000 C CNN
 F 1 "testpoint_cutline" H 2300 2200 50  0001 C CNN
-F 2 "WM1200:testpoint_cutline" H 2450 2050 50  0001 C CNN
+F 2 "WM1200:testpoint_cutline_fat" H 2450 2050 50  0001 C CNN
 F 3 "" H 2450 2050 50  0001 C CNN
 	1    2300 2050

Commit message: Some more work done
I'm too lazy to think about commit messages in my pet project, really
Connections:
- net FPGA_VCC5V renamed FPGA_VCC5V_2
Changed lines of the file:
@@
 +3V3_BUFFER
 Text GLabel 6400 4500 2    50   BiDi ~ 0
-FPGA_VCC5V
+FPGA_VCC5V_2
 $EndSCHEMATC

Commit message: board updated - factory DRC checking in progress
Parts:
- JP1: footprint Connector_PinHeader_2.54mm:PinHeader_1x03_P2.54mm_Vertical -> WM1200:PinHeader_1x03_P2.54mm_Vertical
- JP2: footprint Connector_PinHeader_2.54mm:PinHeader_1x02_P2.54mm_Vertical -> WM1200:PinHeader_1x02_P2.54mm_Vertical
Changed lines of the file:
@@
 F 0 "JP1" V 3854 3602 50  0000 L CNN
 F 1 "Jumper_NC_Dual" V 3945 3602 50  0000 L CNN
-F 2 "Connector_PinHeader_2.54mm:PinHeader_1x03_P2.54mm_Vertical" H 3900 3500 50  0001 C CNN
+F 2 "WM1200:PinHeader_1x03_P2.54mm_Vertical" H 3900 3500 50  0001 C CNN
 F 3 "~" H 3900 3500 50  0001 C CNN
 	1    3900 3500
@@
 F 0 "JP2" H 3900 4764 50  0000 C CNN
 F 1 "Jumper" H 3900 4673 50  0000 C CNN
-F 2 "Connector_PinHeader_2.54mm:PinHeader_1x02_P2.54mm_Vertical" H 3900 4500 50  0001 C CNN
+F 2 "WM1200:PinHeader_1x02_P2.54mm_Vertical" H 3900 4500 50  0001 C CNN
 F 3 "~" H 3900 4500 50  0001 C CNN
 	1    3900 4500
